File: kicad_project/attnode_v3_micro.kicad_pcb (KiCad board)
At the start: 2 copper layers, 16 x 16 mm, 14 parts, among them J1 Conn_01x08_Male, J2 Conn_01x08_Male, J3 Conn_01x04_Male, U1 ATtiny3216-S

Commit message: update readme
Other:
- board text added: "J1"
- board text added: "J2"
- board text added: "µ-attno.de V3.0"
- board text removed: "µ-attno.de V3"
Changed lines of the file:
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@@
   (general
     (thickness 1.6)
-    (drawings 10)
+    (drawings 14)
     (tracks 103)
     (zones 0)
@@
     (38 B.Mask user)
     (39 F.Mask user)
-    (40 Dwgs.User user)
-    (41 Cmts.User user)
-    (42 Eco1.User user)
-    (43 Eco2.User user)
-    (44 Edge.Cuts user)
-    (45 Margin user)
-    (46 B.CrtYd user)
-    (47 F.CrtYd user)
-    (48 B.Fab user)
-    (49 F.Fab user)
+    (40 Dwgs.User user hide)
+    (41 Cmts.User user hide)
+    (42 Eco1.User user hide)
+    (43 Eco2.User user hide)
+    (44 Edge.Cuts user hide)
+    (45 Margin user hide)
+    (46 B.CrtYd user hide)
+    (47 F.CrtYd user hide)
+    (48 B.Fab user hide)
+    (49 F.Fab user hide)
   )
   (setup
@@
     (mod_text_size 1 1)
     (mod_text_width 0.15)
-    (pad_size 1 1)
+    (pad_size 2.5 1.5)
     (pad_drill 0)
     (pad_to_mask_clearance 0)
@@
       (effects (font (size 1 1) (thickness 0.15)) (justify mirror))
     )
-    (pad 1 smd roundrect (at 0 0 270) (size 2.5 1.5) (layers B.Cu B.Paste B.Mask) (roundrect_rratio 0.067)
+    (pad 1 smd roundrect (at 0 0 270) (size 2.5 1.5) (layers B.Cu B.Mask) (roundrect_rratio 0.067)
       (net 7 RST))
   )
@@
       (effects (font (size 1 1) (thickness 0.15)) (justify mirror))
     )
-    (pad 1 smd roundrect (at 0 0 270) (size 2.5 1.5) (layers B.Cu B.Paste B.Mask) (roundrect_rratio 0.067)
+    (pad 1 smd roundrect (at 0 0 270) (size 2.5 1.5) (layers B.Cu B.Mask) (roundrect_rratio 0.067)
       (net 14 RX))
   )
@@
       (effects (font (size 1 1) (thickness 0.15)) (justify mirror))
     )
-    (pad 1 smd roundrect (at 0 0 270) (size 2.5 1.5) (layers B.Cu B.Paste B.Mask) (roundrect_rratio 0.067)
+    (pad 1 smd roundrect (at 0 0 270) (size 2.5 1.5) (layers B.Cu B.Mask) (roundrect_rratio 0.067)
       (net 13 TX))
   )
@@
     (descr "Through hole straight pin header, 1x04, 2.54mm pitch, single row")
     (tags "Through hole pin header THT 1x04 2.54mm single row")
-    (fp_text reference J3 (at 0.19 1.73 -90) (layer B.SilkS)
+    (fp_text reference J3 (at 0.01 1.54 -90) (layer B.SilkS)
       (effects (font (size 0.9 0.9) (thickness 0.09)) (justify mirror))
     )
@@
     (fp_line (start 1.8 -9.4) (end 1.8 1.8) (layer B.CrtYd) (width 0.05))
     (fp_line (start 1.8 1.8) (end -1.8 1.8) (layer B.CrtYd) (width 0.05))
-    (fp_text user %R (at 0 -3.81) (layer B.Fab)
-      (effects (font (size 1 1) (thickness 0.15)) (justify mirror))
+    (fp_text user %R (at 0.89 -9.02) (layer F.SilkS)
+      (effects (font (size 0.6 0.6) (thickness 0.07)))
     )
     (pad 4 thru_hole oval (at 0 -7.62 90) (size 1.7 1.7) (drill 1) (layers *.Cu *.Mask)
@@
     (attr smd)
     (fp_text reference U1 (at -0.09 -7.04) (layer F.SilkS)
-      (effects (font (size 0.7 0.7) (thickness 0.07)))
+      (effects (font (size 0.6 0.6) (thickness 0.07)))
     )
     (fp_text value ATtiny3216-S (at 0 7.35) (layer F.Fab)
@@
     (descr "Through hole straight pin header, 1x08, 2.00mm pitch, single row")
     (tags "Through hole pin header THT 1x08 2.00mm single row")
-    (fp_text reference J1 (at 0 -2.06) (layer F.SilkS) hide
-      (effects (font (size 1 1) (thickness 0.15)))
+    (fp_text reference J1 (at -1.98 14.1) (layer B.SilkS)
+      (effects (font (size 0.75 0.75) (thickness 0.08)) (justify mirror))
     )
     (fp_text value Conn_01x08_Male (at 0 16.06) (layer F.Fab) hide
@@
     (descr "Through hole straight pin header, 1x08, 2.00mm pitch, single row")
     (tags "Through hole pin header THT 1x08 2.00mm single row")
-    (fp_text reference J2 (at 0 -2.06) (layer F.SilkS) hide
-      (effects (font (size 1 1) (thickness 0.15)))
+    (fp_text reference J2 (at 1.83 14.05) (layer B.SilkS)
+      (effects (font (size 0.75 0.75) (thickness 0.08)) (justify mirror))
     )
     (fp_text value Conn_01x08_Male (at 0 16.06) (layer F.Fab) hide
@@
     )
   )
+  (gr_text J2 (at 63.71 65.04 90) (layer F.SilkS)
+    (effects (font (size 0.6 0.6) (thickness 0.07)))
+  )
+  (gr_text J1 (at 52.32 65.05 90) (layer F.SilkS)
+    (effects (font (size 0.6 0.6) (thickness 0.07)))
+  )
+  (gr_circle (center 52.12 50.73) (end 52.198102 50.73) (layer B.SilkS) (width 0.12))
+  (gr_circle (center 69.361898 60.43) (end 69.44 60.43) (layer B.SilkS) (width 0.12))
   (gr_circle (center 63.54 62.31) (end 63.49 62.37) (layer F.SilkS) (width 0.12))
   (gr_circle (center 52.12 50.73) (end 52.07 50.79) (layer F.SilkS) (width 0.12))
@@
     (effects (font (size 0.5 0.5) (thickness 0.07)) (justify mirror))
   )
-  (gr_text "µ-attno.de V3" (at 52.79 55.43 90) (layer B.SilkS)
+  (gr_text "µ-attno.de \nV3.0" (at 53.38 57.27 90) (layer B.SilkS)
     (effects (font (size 0.9 0.9) (thickness 0.1)) (justify mirror))
   )
